Commit message: 修正kinect模型的外观

File: src/jackal_description/urdf/accessories/kinect.urdf.xacro (robot description, xacro)
@@ -7,5 +7,5 @@
             <origin xyz="0 0 0" rpy="0 0 0"/>
             <visual>
-                <origin xyz="0 0 0" rpy="0 0 ${M_PI/2}"/>
+                <origin xyz="0 0 0" rpy="0 0 0"/>
                 <geometry>
                     <mesh filename="package://jackal_description/meshes/kinect.dae" scale="0.4 0.4 0.4" />
