Commit message: add kinect

File: src/jackal_description/urdf/accessories.urdf.xacro (robot description, xacro)
@@ -255,4 +255,5 @@
     - JACKAL_STEREO_FLEA3
     - JACKAL_BB2
+    - Kinect
   -->
   <!-- Common camera mounts and accessory URDFs. -->
@@ -260,5 +261,5 @@
   <xacro:include filename="$(find pointgrey_camera_description)/urdf/pointgrey_flea3.urdf.xacro" />
   <!-- If enabled, generate the flea3 camera payload with a tilt of 30 degrees. -->
-  <xacro:if value="$(optenv JACKAL_FLEA3 1)">
+  <xacro:if value="$(optenv JACKAL_FLEA3 0)">
     <xacro:property name="name" value="$(optenv JACKAL_FLEA3_NAME front)" />
     <xacro:property name="tilt" value="$(optenv JACKAL_FLEA3_TILT 0.)" />
@@ -380,4 +381,45 @@
     </xacro:unless>
   </xacro:if>
+  <xacro:if value="$(optenv KINECT 1)">
+    <xacro:property name="name" value="$(optenv KINECT_NAME front)" />
+    <xacro:property name="tilt" value="$(optenv KINECT_TILT 0.)" />
+    <xacro:property name="tower" value="$(optenv KINECT_TOWER 1)" />
+    <xacro:property name="mount" value="$(optenv KINECT_MOUNT front)" />
+    <xacro:property name="prefix" value="$(optenv KINECT_PREFIX ${mount})" />
+    <xacro:property name="parent" value="$(optenv KINECT_PARENT ${mount}_mount)" />
+    <xacro:include filename="$(find jackal_description)/urdf/accessories/kinect.urdf.xacro"/>
+    <xacro:kinect_camera prefix="front"/>
+    <!-- Mount Enabled -->
+    <xacro:if value="${tower}">
+      <xacro:camera_mount prefix="${prefix}" tilt="${tilt}"/>
+      <joint name="${prefix}_camera_mount_joint" type="fixed">
+        <origin xyz="$(optenv JACKAL_KINECT_OFFSET 0 0 0)"
+                rpy="$(optenv JACKAL_KINECT_RPY 0 0 0)" />
+        <parent link="${parent}" />
+        <child link="${prefix}_camera_mount" />
+      </joint>
+      <joint name="${prefix}_camera_bracket_joint" type="fixed">
+        <origin xyz="0.020 0 0.0245" rpy="0 0 0" />
+        <parent link="${prefix}_camera_beam" />
+        <child link="${prefix}_kinect" />
+      </joint>
+    </xacro:if>
+    <!-- Mount Disabled -->
+    <xacro:unless value="${tower}">
+      <link name="${prefix}_camera_base"/>
+      <joint name="${prefix}_camera_base_joint" type="fixed">
+        <origin xyz="$(optenv JACKAL_KINECT_OFFSET 0 0 0)"
+                rpy="$(optenv JACKAL_KINECT_RPY 0 0 0)" />
+        <parent link="${parent}" />
+        <child link="${prefix}_camera_base" />
+      </joint>
+      <joint name="${prefix}_camera_joint" type="fixed">
+        <origin xyz="0 0 0.0145"
+                rpy="0 0 0" />
+        <parent link="${prefix}_camera_base" />
+        <child link="${prefix}_kinect" />
+      </joint>
+    </xacro:unless>
+  </xacro:if>
   <!-- BlackflyS Camera -->
   <xacro:include filename="$(find flir_camera_description)/urdf/flir_blackflys.urdf.xacro"/>

Commit message: add meshes

File: src/jackal_description/urdf/accessories.urdf.xacro (robot description, xacro)
@@ -342,5 +342,5 @@
   <!-- If enabled, generate the bumblebee2 camera payload with a tilt of 0 degrees. -->
   <!-- Disabled temporarily due to metapackage issue. -->
-  <xacro:if value="$(optenv JACKAL_BB2 1)">
+  <xacro:if value="$(optenv JACKAL_BB2 0)">
     <xacro:property name="tilt" value="$(optenv JACKAL_BB2_TILT 0)" />
     <xacro:property name="name" value="$(optenv JACKAL_BB2_NAME front)" />

File: src/jackal_description/urdf/accessories/kinect.urdf.xacro (robot description, xacro)
@@ -9,5 +9,5 @@
                 <origin xyz="0 0 0" rpy="0 0 ${M_PI/2}"/>
                 <geometry>
-                    <mesh filename="package://turtlebot3_description/meshes/kinect.dae" scale="0.4 0.4 0.4" />
+                    <mesh filename="package://jackal_description/meshes/kinect.dae" scale="0.4 0.4 0.4" />
                 </geometry>
             </visual>

Commit message: model update

File: src/jackal_description/urdf/accessories.urdf.xacro (robot description, xacro)
@@ -400,5 +400,5 @@
       </joint>
       <joint name="${prefix}_camera_bracket_joint" type="fixed">
-        <origin xyz="0.020 0 0.0245" rpy="0 0 0" />
+        <origin xyz="0.020 0 -0.0245" rpy="0 0 0" />
         <parent link="${prefix}_camera_beam" />
         <child link="${prefix}_kinect" />
